File: cpm_vehicle_pcb.kicad_pcb (KiCad board)
At the start: 2 copper layers, 71 parts, among them IC1 ATMEGAAU, IC2 RPI-ZERO, J1 Conn_02x03_Counter_Clockwise, J2 Conn_02x03_Counter_Clockwise, J3 Conn_01x05, J5 USB_B_Mini, J6 Conn_01x03_Socket, P1 NCP1117, Q11 BSS123, Q12 BSS123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

Commit message: update
Parts:
- added J4: USB4105-GF-A, footprints_vehicle_pcb:GCT_USB4105-GF-A, F.Cu at (173.1, 43.0)
- moved L1 0.86 mm to (173.0, 54.5)

Commit message: Routing 2
Parts:
- moved R11 15.4 mm to (128.8, 70.7), turned to 180 degrees
- moved R15 10.9 mm to (111.0, 88.4)
- moved R14 10.9 mm to (128.8, 63.1), turned to 180 degrees
- moved Q11 10.5 mm to (111.0, 84.3)
- moved R13 7.34 mm to (128.8, 61.5), turned to 180 degrees
- moved C42 7.31 mm to (118.8, 61.7)
- moved R16 7.11 mm to (100.1, 88.4)
- moved R18 6.92 mm to (105.1, 83.3)
- moved Q12 6.61 mm to (103.2, 78.9)
- moved C53 6.42 mm to (156.4, 49.9), turned to 180 degrees
- moved Q14 6.16 mm to (111.1, 78.0)
- moved C51 3.92 mm to (137.5, 50.8)
- moved R12 2.58 mm to (128.8, 59.9), turned to 180 degrees
- moved C54 1.74 mm to (133.0, 50.8), turned to 180 degrees
- moved Q13 1.26 mm to (107.2, 78.9)
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Connections:
- J1 pad 3: /LED1_PIN -> /LED2_PIN
- J1 pad 4: /LED2_PIN -> /LED4_PIN
- J1 pad 5: /LED4_PIN -> /LED1_PIN
- J3 pad 1: /SERVO_PWM -> /PWM
- J3 pad 5: /PWM -> /SERVO_PWM
Routing:
- net +5V: track 64.1 -> 229.7 mm, vias 0 -> 5
- net /ERW5: track 0.00 -> 48.9 mm, vias 0 -> 1
- net /MODE: track 0.00 -> 43.5 mm
- net /R12: track 0.00 -> 31.3 mm, vias 0 -> 2
- net /R13: track 0.00 -> 27.5 mm, vias 0 -> 2
- net /PWM: track 0.00 -> 26.7 mm, vias 0 -> 1
- net /RX0: track 0.00 -> 24.6 mm, vias 0 -> 2
- net /TX0: track 0.00 -> 24.6 mm, vias 0 -> 2
- net /R11: track 0.00 -> 23.7 mm
- net /R14: track 0.00 -> 22.5 mm, vias 0 -> 2
- net /SERVO_PWM: track 0.91 -> 23.3 mm, vias 0 -> 1
- net GND: track 0.39 -> 13.3 mm, vias 4 -> 7
- net /R15: track 9.25 -> 2.17 mm
- net /LED1: track 0.00 -> 6.06 mm
- net /LED2: track 0.00 -> 5.96 mm
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