File: cpm_vehicle_pcb.kicad_pcb (KiCad board)
At the start: 2 copper layers, 95 x 50 mm, 80 parts, among them IC1 ATMEGAAU, IC2 RPI-ZERO, J1 Conn_02x03_Counter_Clockwise, J2 Conn_02x03_Counter_Clockwise, J3 Conn_01x05, J4 USB3090-XX-X_REVE2, J5 USB_B_Mini, J6 Conn_01x03_Socket, P1 NCP1117, Q11 BSS123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

Commit message: FinalV_1
Parts:
- added R21: 20k, Resistor_SMD:R_0603_1608Metric, F.Cu at (104.3, 63.7)
- added R8: 47k, Resistor_SMD:R_0603_1608Metric, F.Cu at (165.1, 90.1)
- SW1: footprint Button_Switch_SMD:SW_DIP_SPSTx02_Slide_9.78x7.26mm_W8.61mm_P2.54mm -> Button_Switch_SMD:SW_DIP_SPSTx01_Slide_9.78x4.72mm_W8.61mm_P2.54mm
- SW2: value SW_SPST -> SW_DPDT_x2
- moved C31 7.08 mm to (98.8, 50.5), turned to 180 degrees
- moved C41 4.90 mm to (120.2, 63.8), turned to 90 degrees
- moved C42 4.51 mm to (123.1, 60.5)
- moved SW2 0.13 mm to (169.2, 87.5), turned to 180 degrees
- turned SW1 to 0 degrees
Connections:
- SW2 pad 2: vcc_bat -> unconnected-(SW2A-A-Pad2)
- SW2 pad 3: (no net) -> vcc_bat
Routing:
- net Net-(U3-OE): track 0.00 -> 51.8 mm, vias 0 -> 2
- net +3V3: track 81.5 -> 47.5 mm
- net +5V: track 269.6 -> 288.4 mm
- net (no net): track 16.4 -> 0.00 mm
- net vcc_bat: track 28.5 -> 30.2 mm, vias 1 -> 0
- net B+: track 54.2 -> 55.3 mm
- net GND: vias 10 -> 13
