File: _autosave-cpm_vehicle_pcb.kicad_sch (KiCad schematic)
At the start: 82 parts, among them IC1 ATMEGAAU, IC2 RPI-ZERO, J1 Conn_02x03_Counter_Clockwise, J2 Conn_02x03_Counter_Clockwise, J3 Conn_01x05, J5 USB_B_Mini, J6 Conn_01x03_Socket, P1 NCP1117, Q11 BSS123, Q12 BSS123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

Commit message: Ver2
Parts:
- USB1: footprint Connector_USB:USB_C_Receptacle_HRO_TYPE-C-31-M-17 -> footprints_vehicle_pcb:USB-C-SMD_10P-P1.00-L6.8-W8.9
Changed lines of the file:
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@@
 			)
 		)
-		(property "Footprint" "Connector_USB:USB_C_Receptacle_HRO_TYPE-C-31-M-17"
+		(property "Footprint" "footprints_vehicle_pcb:USB-C-SMD_10P-P1.00-L6.8-W8.9"
 			(at 154.94 21.59 0)
 			(effects
